Commit message: added fixex from review

File: my_rb1_description/urdf/my_rb1_robot.urdf (robot description, URDF)
Before this commit: robot robot, 7 links, 6 joints
Joints:
- joint joint_left_wheel_link: limit effort=1000 velocity=1000 -> effort=10000 velocity=1000
- joint joint_right_wheel_link: limit effort=1000 velocity=1000 -> effort=10000 velocity=1000

Commit message: changed urdf file

File: my_rb1_description/urdf/my_rb1_robot.urdf (robot description, URDF)
Before this commit: robot robot, 7 links, 6 joints
Joints:
- joint joint_left_wheel_link: limit effort=10000 velocity=1000 -> (none)
- joint joint_right_wheel_link: limit effort=10000 velocity=1000 -> (none)
